File: final.kicad_pcb (KiCad board)
At the start: 2 copper layers, 231.5 x 118.4 mm, 79 parts

Commit message: wip
Routing:
- net P2: track 0.00 -> 275.6 mm
- net P21: track 0.00 -> 234.5 mm
- net P8: track 0.00 -> 232.9 mm
- net P16: track 0.00 -> 179.7 mm
- net P4: track 0.00 -> 175.9 mm
- net P19: track 0.00 -> 175.4 mm
- net P5: track 0.00 -> 148.7 mm
- net P18: track 0.00 -> 148.7 mm
- net P3: track 0.00 -> 143.5 mm
- net P20: track 0.00 -> 142.9 mm
- net P6: track 0.00 -> 126.9 mm
- net P15: track 0.00 -> 126.5 mm
- net P7: track 0.00 -> 118.2 mm
- net P14: track 0.00 -> 118.1 mm
- net GND: track 0.00 -> 68.2 mm
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